File: PCB/Hotair-soldering-station/main-pcb/hotair-soldering-station-main-pcb.sch (KiCad schematic (older format))
At the start: 82 parts, among them J2 main-board-conn

Commit message: main pcb smsps fan add
Parts:
- removed D?: 8V2, Diode_THT:D_DO-34_SOD68_P7.62mm_Horizontal, symbol Device:D_Zener
- removed Q?: BD681, TO_SOT_Packages_THT:TO-126_Vertical, symbol Transistor_BJT:TIP122
- removed Q? (x2): BC817, Package_TO_SOT_SMD:SOT-23, symbol Transistor_BJT:BC817
- removed R? (x2): 5k1, Capacitors:0805, symbol Device:R
- removed R?: 10k, Capacitors:0805, symbol Device:R
- removed R?: 5k6, Capacitors:0805, symbol Device:R
- removed R?: 7k5, Capacitors:0805, symbol Device:R
- added C? (x2): 47u/35V, symbol Device:CP
- added C?: 100u/35V, symbol Device:CP
- added C?: 470p, Capacitors:0805, symbol Device:C
- added C?: 1u, Capacitors:0805, symbol Device:C
- added D? (x2): 1N5819, Diode_THT:D_DO-41_SOD81_P10.16mm_Horizontal, symbol Diode:1N5819
- added D?: 1N4148, Diode_THT:D_DO-35_SOD27_P7.62mm_Horizontal, symbol Diode:1N4148
- added L?: 220uH, symbol pspice:INDUCTOR
- added Q?: IRLIZ44N, Package_TO_SOT_THT:TO-220F-3_Vertical, symbol Transistor_FET:IRLIZ44N
- added Q? (x2): BC817, Package_TO_SOT_SMD:SOT-23, symbol Transistor_BJT:BC817
- added Q?: BC807, Package_TO_SOT_SMD:SOT-23, symbol Transistor_BJT:BC807
- added R?: 100R, Capacitors:0805, symbol Device:R
- added R?: 900R, Capacitors:0805, symbol Device:R
- added R?: 4k7, Capacitors:0805, symbol Device:R
Connections:
- net FAN_POT_A is gone; now on net HOTAIR_FAN_DOWN_SW: J2.5 (Pin_5)
- net FAN_POT_B is gone; now on net HOTAIR_FAN_UP_SW: J2.6 (Pin_6)
- net FAN_POT_W is gone; now on net GND: J2.7 (Pin_7)
- net +24V: now also C?.1, Q?.2 (D)
- net +5V: now also D?.2 (A)
- net FAN_SUPPLY: now also C?.1, C?.1, L?.2
- net GND: now also C?.2, C?.2, C?.2, D?.2 (A), Q?.2 (E), Q?.3 (C)
- net HOTAIR_FAN_DOWN_SW: now reaches U?.2 (PF0)
- net HOTAIR_FAN_UP_SW: now reaches U?.3 (PF1)
- net FAN_EN renamed FAN_PWM
- net FAN_PWM: now also R?.1
- new net: C?.1, D?.1 (K), L?.1, Q?.3 (S)
- new net: Q?.1 (G), Q?.2 (E), Q?.2 (E)
- new net: C?.1, D?.2 (A), Q?.1 (B), R?.2
- new net: D?.1 (K), Q?.1 (B), Q?.1 (B), Q?.3 (C), R?.2
- new net: C?.2, R?.1, R?.2
- new net: C?.2, D?.1 (K), Q?.3 (C), R?.1

Commit message: schematc footprint assign, start pcb routing
Parts:
- removed J?: SOLD_IRON_CONN, My-Footprints:Conn-01x05-N25-W5P, symbol Connector_Generic:Conn_01x05
- removed J?: POWER_SUPPLY, symbol Connector_Generic:Conn_01x02
- added J10: PA11, My-Footprints:WIRE_PAD_1,3mm, symbol Connector_Generic:Conn_01x01
- added J11: PA12, My-Footprints:WIRE_PAD_1,3mm, symbol Connector_Generic:Conn_01x01
- added J12: PA15, My-Footprints:WIRE_PAD_1,3mm, symbol Connector_Generic:Conn_01x01
- added J5: PSUPPLY (PWZ-02S r.3,96), Connectors_Hirose:Hirose_DF63-3P-3.96DSA_03x3.96mm_Straight, symbol Connector_Generic:Conn_01x03
- added J9: SOLD_IRON (r.2,54), My-Footprints:Conn-01x06-N25-W6P, symbol Connector_Generic:Conn_01x06
- added R14, R9: 390R, Resistor_THT:R_Axial_DIN0414_L11.9mm_D4.5mm_P20.32mm_Horizontal, symbol Device:R
- C3: renamed from C?; footprint (none) -> Capacitor_THT:CP_Radial_D10.0mm_P3.80mm
- C5: renamed from C?; footprint (none) -> Capacitor_THT:C_Rect_L13.0mm_W5.0mm_P10.00mm_FKS3_FKP3_MKS4
- C6: renamed from C?; footprint Capacitors:0805 -> Capacitors:1206
- C8, C9: renamed from C?; footprint (none) -> Capacitor_THT:CP_Radial_D6.3mm_P2.50mm
- D1: renamed from D?; value 1N5819 -> MBR052; footprint Diode_THT:D_DO-41_SOD81_P10.16mm_Horizontal -> Diodes_SMD:D_SOD-123
- D2: renamed from D?; footprint Diode_THT:D_DO-35_SOD27_P7.62mm_Horizontal -> Diodes_SMD:D_MiniMELF
- F1, F2, F3: renamed from F?; footprint (none) -> Fuse_Holders_and_Fuses:Fuseholder5x20_horiz_SemiClosed_Casing10x25mm
- J1: renamed from J?; footprint (none) -> My-Footprints:Screw-Terminal-5.00mm-3pin
- J13: renamed from J?; value ICP -> ICP (goldpin r2,54)
- J3: renamed from J?; footprint (none) -> My-Footprints:Screw-Terminal-5.00mm-2pin
- J4: renamed from J?; value 24V_IN -> 24V_IN (NS-25 r2,54); footprint (none) -> My-Footprints:Conn-01x04-N25-W4P
- J6: renamed from J?; value HOTAIR_FAN -> HOTAIR_FAN (JST r,2,54)
- J7: renamed from J?; value HOTAIR_MEAS -> HOTAIR_MEAS (JST r.2,5)
- J8: renamed from J?; value HOTAIR_HEATER -> HOTAIR_HEATER (PWZ-02S r.3,96)
- L1: renamed from L?; footprint (none) -> Inductors_THT:L_Radial_D10.0mm_P5.00mm_Fastron_07M
- R10: renamed from R?; value 150R -> 390R; footprint Capacitors:0805 -> Resistor_THT:R_Axial_DIN0414_L11.9mm_D4.5mm_P20.32mm_Horizontal
- R12, R17: renamed from R?; footprint Capacitors:0805 -> Resistor_THT:R_Axial_DIN0414_L11.9mm_D4.5mm_P20.32mm_Horizontal
- R15: renamed from R?; value 160R -> 390R; footprint Capacitors:0805 -> Resistor_THT:R_Axial_DIN0414_L11.9mm_D4.5mm_P20.32mm_Horizontal
- R4: renamed from R?; value 900R -> 910R
- U2: renamed from U?; footprint (none) -> Housings_SOIC:SOIC-14_3.9x8.7mm_Pitch1.27mm
- gave numbers to parts that had none: 59
Connections:
- net +24V: now also J9.1 (Pin_1)
- net 7SEG_CLK: now also J2.12 (Pin_12); no longer J2.3 (Pin_3)
- net 7SEG_DIN: now also J2.14 (Pin_14); no longer J2.2 (Pin_2)
- net 7SEG_LATCH: now also J2.13 (Pin_13); no longer J2.4 (Pin_4)
- net AC_230(N): now also J5.2 (Pin_2), J5.3 (Pin_3)
- net GND: now also J2.2 (Pin_2), J2.3 (Pin_3), J9.5 (Pin_5), J9.6 (Pin_6); no longer J2.7 (Pin_7), J2.8 (Pin_8)
- net HOTAIR_DOWN_SW: now also J2.6 (Pin_6); no longer J2.13 (Pin_13)
- net HOTAIR_FAN_DOWN_SW: now also J2.9 (Pin_9); no longer J2.5 (Pin_5)
- net HOTAIR_FAN_UP_SW: now also J2.8 (Pin_8); no longer J2.6 (Pin_6)
- net HOTAIR_UP_SW: now also J2.7 (Pin_7); no longer J2.14 (Pin_14)
- net SOLDERING_IRON_HEATER: now also J9.2 (Pin_2)
- net SOLDERING_IRON_THERM: now also J9.3 (Pin_3)
- net SOLDER_DOWN_SW: now also J2.4 (Pin_4); no longer J2.11 (Pin_11)
- net SOLDER_ON_SW: now also J2.11 (Pin_11); no longer J2.9 (Pin_9)
- net SOLDER_UP_SW: now also J2.5 (Pin_5); no longer J2.12 (Pin_12)
- net at C5.1, R10.2, R15.1: now also R14.1, R9.2
- net at R10.1, U1.6: now also R9.1
- net at J8.1 (Pin_1), Q6.2 (A2), R15.2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: now also R14.2
- net at R26.2: now also J9.4 (Pin_4)
- net at F1.1: now also J5.1 (Pin_1)
- net at U5.21 (PA11): now also J10.1 (Pin_1)
- net at U5.22 (PA12): now also J11.1 (Pin_1)
- net at U5.25 (PA15): now also J12.1 (Pin_1)
Other:
- note added: "2x390R"
- note added: "Power supply for\n230 -> 24V"
