File: PCB/Hotair-soldering-station/main-pcb/hotair-soldering-station-main-pcb.sch (KiCad schematic (older format))
At the start: 90 parts, among them J1 230VAC_IN, J10 PA11, J11 PA12, J12 PA15, J13 ICP (goldpin r2,54), J2 main-board-conn, J3 EARTH_GND, J4 24V_IN (NS-25 r2,54), J5 PSUPPLY (PWZ-02S r.3,96), J6 HOTAIR_FAN (JST r,2,54)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

Commit message: main pcb routing
Parts:
- removed R14, R9: 390R, Resistor_THT:R_Axial_DIN0414_L11.9mm_D4.5mm_P20.32mm_Horizontal, symbol Device:R
- removed U4: AMS1117-3.3, Package_TO_SOT_SMD:SOT-223-3_TabPin2, symbol Regulator_Linear:AMS1117-3.3
- added R33, R34: 100R, Capacitors:0805, symbol Device:R
- added U4: AP1117-ADJ, Package_TO_SOT_SMD:SOT-223-3_TabPin2, symbol Regulator_Linear:AP1117-ADJ
- R10, R15: value 390R -> 2x390R; footprint Resistor_THT:R_Axial_DIN0414_L11.9mm_D4.5mm_P20.32mm_Horizontal -> Resistor_THT:R_Axial_DIN0414_L11.9mm_D4.5mm_P15.24mm_Horizontal
- R12, R17: footprint Resistor_THT:R_Axial_DIN0414_L11.9mm_D4.5mm_P20.32mm_Horizontal -> Resistor_THT:R_Axial_DIN0414_L11.9mm_D4.5mm_P15.24mm_Horizontal
- U3: symbol My-Lib:MP1584-Step-Down -> hotair-soldering-station-main-pcb-rescue:MP1584-Step-Down-My-Lib
Connections:
- net +3V3: now also R34.1, U4.2 (VO)
- net +5V: now also U4.3 (VI)
- net GND: now also U5.31 (BOOT0), R33.2; no longer C14.2, C15.2
- net at Q8.3 (S), R27.1: now also C14.2, C15.2
- new net: R33.1, R34.2, U4.1 (ADJ)
Other:
- note removed: "2x390R"
- moved on the sheet: C14, C15
Changed lines of the file:
@@
-$EndComp
-$Comp
-L Device:R R15
-U 1 1 5F7F6211
-P 3900 6000
-F 0 "R15" V 3900 6075 50  0000 R CNN
-F 1 "390R" V 3800 6100 50  0001 R CNN
-F 2 "Resistor_THT:R_Axial_DIN0414_L11.9mm_D4.5mm_P20.32mm_Horizontal" V 3830 6000 50  0001 C CNN
-F 3 "~" H 3900 6000 50  0001 C CNN
-	1    3900 6000
-	0    -1   -1   0
 $EndComp
 $Comp
@@
 F 0 "R12" H 3900 6650 50  0000 R CNN
 F 1 "390R" H 4000 6550 50  0000 R CNN
-F 2 "Resistor_THT:R_Axial_DIN0414_L11.9mm_D4.5mm_P20.32mm_Horizontal" V 3680 6600 50  0001 C CNN
+F 2 "Resistor_THT:R_Axial_DIN0414_L11.9mm_D4.5mm_P15.24mm_Horizontal" V 3680 6600 50  0001 C CNN
 F 3 "~" H 3750 6600 50  0001 C CNN
 	1    3750 6600
@@
 	3500 6750 3500 6350
 Connection ~ 3750 6750
-Wire Wire Line
-	3750 6000 3650 6000
 Wire Wire Line
 	3500 6000 3500 6050
@@
 L Device:CP C14
 U 1 1 5F8484E7
-P 11125 7075
-F 0 "C14" H 11243 7121 50  0000 L CNN
-F 1 "330u/35V" H 11243 7030 50  0000 L CNN
-F 2 "Capacitors_THT:CP_Radial_D10.0mm_P5.00mm" H 11163 6925 50  0001 C CNN
-F 3 "~" H 11125 7075 50  0001 C CNN
-	1    11125 7075
+P 11100 6875
+F 0 "C14" H 11218 6921 50  0000 L CNN
+F 1 "330u/35V" H 11218 6830 50  0000 L CNN
+F 2 "Capacitors_THT:CP_Radial_D10.0mm_P5.00mm" H 11138 6725 50  0001 C CNN
+F 3 "~" H 11100 6875 50  0001 C CNN
+	1    11100 6875
 	1    0    0    -1
 $EndComp
@@
 L power:+24V #PWR0114
 U 1 1 5F86C66F
-P 11125 6925
-F 0 "#PWR0114" H 11125 6775 50  0001 C CNN
-F 1 "+24V" H 11140 7098 50  0000 C CNN
-F 2 "" H 11125 6925 50  0001 C CNN
-F 3 "" H 11125 6925 50  0001 C CNN
-	1    11125 6925
-	1    0    0    -1
-$EndComp
-$Comp
-L power:GND #PWR0116
-U 1 1 5F86CA1F
-P 11125 7225
-F 0 "#PWR0116" H 11125 6975 50  0001 C CNN
-F 1 "GND" H 11130 7052 50  0000 C CNN
-F 2 "" H 11125 7225 50  0001 C CNN
-F 3 "" H 11125 7225 50  0001 C CNN
-	1    11125 7225
+P 11100 6725
+F 0 "#PWR0114" H 11100 6575 50  0001 C CNN
+F 1 "+24V" H 11115 6898 50  0000 C CNN
+F 2 "" H 11100 6725 50  0001 C CNN
+F 3 "" H 11100 6725 50  0001 C CNN
+	1    11100 6725
 	1    0    0    -1
 $EndComp
@@
 $EndComp
 Wire Wire Line
-	10175 6975 10175 7175
-Wire Wire Line
-	6500 2825 6500 2725
-$Comp
-L power:GND #PWR0131
-U 1 1 5F9705C8
-P 6500 2825
-F 0 "#PWR0131" H 6500 2575 50  0001 C CNN
-F 1 "GND" H 6505 2652 50  0000 C CNN
-F 2 "" H 6500 2825 50  0001 C CNN
-F 3 "" H 6500 2825 50  0001 C CNN
-	1    6500 2825
-	1    0    0    -1
-$EndComp
-$Comp
-L Regulator_Linear:AMS1117-3.3 U4
-U 1 1 5F87AB31
-P 6500 2425
-F 0 "U4" H 6500 2667 50  0000 C CNN
-F 1 "AMS1117-3.3" H 6500 2576 50  0000 C CNN
-F 2 "Package_TO_SOT_SMD:SOT-223-3_TabPin2" H 6500 2625 50  0001 C CNN
-F 3 "http://www.advanced-monolithic.com/pdf/ds1117.pdf" H 6600 2175 50  0001 C CNN
-	1    6500 2425
-	1    0    0    -1
-$EndComp
+	10175 6975 10175 7025
 Wire Wire Line
 	10175 7475 10175 7625
@@
 $EndComp
 Wire Wire Line
-	6800 2425 7100 2425
+	6800 2425 6950 2425
 Wire Wire Line
 	7100 2425 7100 2275
@@
 	18450 9150 17950 9150
 $Comp
-L My-Lib:MP1584-Step-Down U3
+L hotair-soldering-station-main-pcb-rescue:MP1584-Step-Down-My-Lib U3
 U 1 1 5F823936
 P 4150 2525
@@
 L Device:CP C15
 U 1 1 5FB4124A
-P 11875 7100
-F 0 "C15" H 11993 7146 50  0000 L CNN
-F 1 "330u/35V" H 11993 7055 50  0000 L CNN
-F 2 "Capacitors_THT:CP_Radial_D10.0mm_P5.00mm" H 11913 6950 50  0001 C CNN
-F 3 "~" H 11875 7100 50  0001 C CNN
-	1    11875 7100
+P 11850 6875
+F 0 "C15" H 11968 6921 50  0000 L CNN
+F 1 "330u/35V" H 11968 6830 50  0000 L CNN
+F 2 "Capacitors_THT:CP_Radial_D10.0mm_P5.00mm" H 11888 6725 50  0001 C CNN
+F 3 "~" H 11850 6875 50  0001 C CNN
+	1    11850 6875
 	1    0    0    -1
 $EndComp
@@
 L power:+24V #PWR0148
 U 1 1 5FB41250
-P 11875 6950
-F 0 "#PWR0148" H 11875 6800 50  0001 C CNN
-F 1 "+24V" H 11890 7123 50  0000 C CNN
-F 2 "" H 11875 6950 50  0001 C CNN
-F 3 "" H 11875 6950 50  0001 C CNN
-	1    11875 6950
-	1    0    0    -1
-$EndComp
-$Comp
-L power:GND #PWR0149
-U 1 1 5FB41256
-P 11875 7250
-F 0 "#PWR0149" H 11875 7000 50  0001 C CNN
-F 1 "GND" H 11880 7077 50  0000 C CNN
-F 2 "" H 11875 7250 50  0001 C CNN
-F 3 "" H 11875 7250 50  0001 C CNN
-	1    11875 7250
+P 11850 6725
+F 0 "#PWR0148" H 11850 6575 50  0001 C CNN
+F 1 "+24V" H 11865 6898 50  0000 C CNN
+F 2 "" H 11850 6725 50  0001 C CNN
+F 3 "" H 11850 6725 50  0001 C CNN
+	1    11850 6725
 	1    0    0    -1
 $EndComp
@@
 F 0 "R17" H 4950 6200 50  0000 R CNN
 F 1 "100R" H 5050 6100 50  0000 R CNN
-F 2 "Resistor_THT:R_Axial_DIN0414_L11.9mm_D4.5mm_P20.32mm_Horizontal" V 4730 6150 50  0001 C CNN
+F 2 "Resistor_THT:R_Axial_DIN0414_L11.9mm_D4.5mm_P15.24mm_Horizontal" V 4730 6150 50  0001 C CNN
 F 3 "~" H 4800 6150 50  0001 C CNN
 	1    4800 6150
 	1    0    0    -1
 $EndComp
-$Comp
-L Device:R R9
-U 1 1 5FB374AD
-P 3250 5875
-F 0 "R9" V 3250 5950 50  0000 R CNN
-F 1 "390R" V 3150 5975 50  0001 R CNN
-F 2 "Resistor_THT:R_Axial_DIN0414_L11.9mm_D4.5mm_P20.32mm_Horizontal" V 3180 5875 50  0001 C CNN
-F 3 "~" H 3250 5875 50  0001 C CNN
-	1    3250 5875
-	0    -1   -1   0
-$EndComp
-Wire Wire Line
-	3100 5875 3050 5875
-Wire Wire Line
-	3050 5875 3050 6000
-Connection ~ 3050 6000
-Wire Wire Line
-	3400 5875 3500 5875
-Wire Wire Line
-	3500 5875 3500 6000
-$Comp
-L Device:R R14
-U 1 1 5FB72A06
-P 3900 5875
-F 0 "R14" V 3900 5950 50  0000 R CNN
-F 1 "390R" V 3800 5975 50  0001 R CNN
-F 2 "Resistor_THT:R_Axial_DIN0414_L11.9mm_D4.5mm_P20.32mm_Horizontal" V 3830 5875 50  0001 C CNN
-F 3 "~" H 3900 5875 50  0001 C CNN
-	1    3900 5875
-	0    -1   -1   0
-$EndComp
-Wire Wire Line
-	4050 5875 4150 5875
-Wire Wire Line
-	4150 5875 4150 6000
-Wire Wire Line
-	3750 5875 3650 5875
-Wire Wire Line
-	3650 5875 3650 6000
-Connection ~ 3650 6000
-Wire Wire Line
-	3650 6000 3500 6000
 $Comp
 L Device:R R10
 U 1 1 5F7D0189
 P 3250 6000
-F 0 "R10" V 3250 6075 50  0000 R CNN
-F 1 "390R" V 3150 6100 50  0001 R CNN
-F 2 "Resistor_THT:R_Axial_DIN0414_L11.9mm_D4.5mm_P20.32mm_Horizontal" V 3180 6000 50  0001 C CNN
+F 0 "R10" V 3325 6075 50  0000 R CNN
+F 1 "2x390R" V 3150 6150 50  0000 R CNN
+F 2 "Resistor_THT:R_Axial_DIN0414_L11.9mm_D4.5mm_P15.24mm_Horizontal" V 3180 6000 50  0001 C CNN
 F 3 "~" H 3250 6000 50  0001 C CNN
 	1    3250 6000
 	0    -1   -1   0
 $EndComp
-Text Notes 3100 5800 0    50   ~ 0
-2x390R
-Text Notes 3750 5800 0    50   ~ 0
-2x390R
 $Comp
 L Connector_Generic:Conn_01x01 J10
@@
 P 19150 9250
 F 0 "J10" H 19225 9250 50  0000 L CNN
-F 1 "PA11" H 19350 9250 50  0000 L CNN
+F 1 "PA11" H 19400 9250 50  0000 L CNN
 F 2 "My-Footprints:WIRE_PAD_1,3mm" H 19150 9250 50  0001 C CNN
 F 3 "~" H 19150 9250 50  0001 C CNN
@@
 P 19150 9350
 F 0 "J11" H 19225 9350 50  0000 L CNN
-F 1 "PA12" H 19350 9350 50  0000 L CNN
+F 1 "PA12" H 19400 9350 50  0000 L CNN
 F 2 "My-Footprints:WIRE_PAD_1,3mm" H 19150 9350 50  0001 C CNN
 F 3 "~" H 19150 9350 50  0001 C CNN
@@
 P 19150 9650
 F 0 "J12" H 19225 9650 50  0000 L CNN
-F 1 "PA15" H 19350 9650 50  0000 L CNN
+F 1 "PA15" H 19400 9650 50  0000 L CNN
 F 2 "My-Footprints:WIRE_PAD_1,3mm" H 19150 9650 50  0001 C CNN
 F 3 "~" H 19150 9650 50  0001 C CNN
@@
 Wire Wire Line
 	19100 3000 19100 3425
+$Comp
+L power:GND #PWR0116
+U 1 1 5FA8FEE8
+P 16700 8475
+F 0 "#PWR0116" H 16700 8225 50  0001 C CNN
+F 1 "GND" H 16705 8302 50  0000 C CNN
+F 2 "" H 16700 8475 50  0001 C CNN
+F 3 "" H 16700 8475 50  0001 C CNN
+	1    16700 8475
+	1    0    0    -1
+$EndComp
+Wire Wire Line
+	16850 8350 16700 8350
+Wire Wire Line
+	16700 8350 16700 8475
+Wire Wire Line
+	10175 7025 11100 7025
+Connection ~ 10175 7025
+Wire Wire Line
+	10175 7025 10175 7175
+Connection ~ 11100 7025
+Wire Wire Line
+	11100 7025 11850 7025
+$Comp
+L Regulator_Linear:AP1117-ADJ U4
+U 1 1 5FBD0655
+P 6500 2425
+F 0 "U4" H 6500 2667 50  0000 C CNN
+F 1 "AP1117-ADJ" H 6500 2576 50  0000 C CNN
+F 2 "Package_TO_SOT_SMD:SOT-223-3_TabPin2" H 6500 2625 50  0001 C CNN
+F 3 "http://www.diodes.com/datasheets/AP1117.pdf" H 6600 2175 50  0001 C CNN
+	1    6500 2425
+	1    0    0    -1
+$EndComp
+$Comp
+L Device:R R33
+U 1 1 5FBD0F67
+P 6500 3050
+F 0 "R33" V 6425 3100 50  0000 R CNN
+F 1 "100R" V 6575 3150 50  0000 R CNN
+F 2 "Capacitors:0805" V 6430 3050 50  0001 C CNN
+F 3 "~" H 6500 3050 50  0001 C CNN
+	1    6500 3050
+	1    0    0    -1
+$EndComp
+$Comp
+L Device:R R34
+U 1 1 5FC0C3F0
+P 6725 2875
+F 0 "R34" V 6650 2925 50  0000 R CNN
+F 1 "100R" V 6800 2975 50  0000 R CNN
+F 2 "Capacitors:0805" V 6655 2875 50  0001 C CNN
+F 3 "~" H 6725 2875 50  0001 C CNN
+	1    6725 2875
+	0    1    1    0
+$EndComp
+Wire Wire Line
+	6875 2875 6950 2875
+Wire Wire Line
+	6950 2875 6950 2425
+Connection ~ 6950 2425
+Wire Wire Line
+	6950 2425 7100 2425
+Wire Wire Line
+	6575 2875 6500 2875
+Wire Wire Line
+	6500 2725 6500 2875
+Wire Wire Line
+	6500 2875 6500 2900
+Connection ~ 6500 2875
+$Comp
+L power:GND #PWR0131
+U 1 1 5FC69697
+P 6500 3200
+F 0 "#PWR0131" H 6500 2950 50  0001 C CNN
+F 1 "GND" H 6505 3027 50  0000 C CNN
+F 2 "" H 6500 3200 50  0001 C CNN
+F 3 "" H 6500 3200 50  0001 C CNN
+	1    6500 3200
+	1    0    0    -1
+$EndComp
+Wire Wire Line
+	3500 6000 3750 6000
+$Comp
+L Device:R R15
+U 1 1 5F7F6211
+P 3900 6000
+F 0 "R15" V 3975 6075 50  0000 R CNN
+F 1 "2x390R" V 3800 6125 50  0000 R CNN
+F 2 "Resistor_THT:R_Axial_DIN0414_L11.9mm_D4.5mm_P15.24mm_Horizontal" V 3830 6000 50  0001 C CNN
+F 3 "~" H 3900 6000 50  0001 C CNN
+	1    3900 6000
+	0    -1   -1   0
+$EndComp
 $EndSCHEMATC

Commit message: PCB desingn update
Parts:
- removed R11, R26: 0R, Capacitors:0805, symbol Device:R
- added R9: 0R, Capacitors:0805, symbol Device:R
- D3: footprint Diode_THT:D_DO-41_SOD81_P10.16mm_Horizontal -> Diode_SMD:D_MELF
- Q6: footprint Package_TO_SOT_THT:TO-220-3_Vertical -> My-Footprints:TO-220-3_Vertical
Connections:
- net +24V: now also J9.2 (Pin_2)
- net GND: now also R9.2; no longer J9.5 (Pin_5), J9.6 (Pin_6)
- net SOLDERING_IRON_THERM: now also J9.5 (Pin_5); no longer J9.3 (Pin_3)
- net at C4.2, R5.2, R7.1: now also U2.6 (-); no longer U2.9 (-)
- net at C4.1, R7.2: now also U2.10 (+), U2.7; no longer U2.5 (+), U2.8
- net at C1.1, R2.2: now also U2.5 (+); no longer U2.10 (+)
- net at R16.2, R18.1: now also U2.8; no longer U2.7
- net THERM_GND: now reaches J7.2 (Pin_2)
- net THERM_GND: now also J9.6 (Pin_6), R9.1
- net at R13.2, R16.1: now also U2.9 (-); no longer U2.6 (-)
- net SOLDERING_IRON_HEATER_GND: now reaches J9.4 (Pin_4)
- net SOLDERING_IRON_HEATER_GND: now also J9.3 (Pin_3), Q8.2 (D)
- removed net SOLDERING_IRON_HEATER: J9.2 (Pin_2), Q8.2 (D)
Other:
- moved on the sheet: U2B, U2C
Changed lines of the file:
@@
 F 0 "Q6" H 4250 6400 39  0000 L CNN
 F 1 "BT139-600" H 4250 6300 39  0000 L CNN
-F 2 "Package_TO_SOT_THT:TO-220-3_Vertical" H 4350 6275 50  0001 L CIN
+F 2 "My-Footprints:TO-220-3_Vertical" H 4350 6275 50  0001 L CIN
 F 3 "https://www.rapidonline.com/pdf/47-3240.pdf" H 4150 6350 50  0001 L CNN
 	1    4150 6350
@@
 L Amplifier_Operational:LMV324 U2
 U 2 1 5F81308B
+P 2800 11900
+F 0 "U2" H 2800 12267 50  0000 C CNN
+F 1 "LMV324" H 2800 12176 50  0000 C CNN
+F 2 "" H 2750 12000 50  0001 C CNN
+F 3 "http://www.ti.com/lit/ds/symlink/lmv324.pdf" H 2850 12100 50  0001 C CNN
+	2    2800 11900
+	1    0    0    1
+$EndComp
+$Comp
+L Amplifier_Operational:LMV324 U2
+U 3 1 5F814694
 P 4425 11800
 F 0 "U2" H 4425 12167 50  0000 C CNN
@@
 F 2 "" H 4375 11900 50  0001 C CNN
 F 3 "http://www.ti.com/lit/ds/symlink/lmv324.pdf" H 4475 12000 50  0001 C CNN
-	2    4425 11800
-	1    0    0    1
-$EndComp
-$Comp
-L Amplifier_Operational:LMV324 U2
-U 3 1 5F814694
-P 2800 11900
-F 0 "U2" H 2800 12267 50  0000 C CNN
-F 1 "LMV324" H 2800 12176 50  0000 C CNN
-F 2 "" H 2750 12000 50  0001 C CNN
-F 3 "http://www.ti.com/lit/ds/symlink/lmv324.pdf" H 2850 12100 50  0001 C CNN
-	3    2800 11900
+	3    4425 11800
 	1    0    0    1
 $EndComp
@@
 	1    0    0    -1
 $EndComp
-$Comp
-L power:GND #PWR0112
-U 1 1 5F812675
-P 10050 12150
-F 0 "#PWR0112" H 10050 11900 50  0001 C CNN
-F 1 "GND" H 10055 11977 50  0000 C CNN
-F 2 "" H 10050 12150 50  0001 C CNN
-F 3 "" H 10050 12150 50  0001 C CNN
-	1    10050 12150
-	1    0    0    -1
-$EndComp
-Wire Wire Line
-	10000 11750 10375 11750
-Wire Wire Line
-	10375 11650 10000 11650
-Text GLabel 10000 11650 0    50   Input ~ 0
-SOLDERING_IRON_HEATER
-Text GLabel 10000 11750 0    50   Input ~ 0
+Text GLabel 9900 11750 0    50   Input ~ 0
+SOLDERING_IRON_HEATER_GND
+Text GLabel 10150 11950 0    50   Input ~ 0
 SOLDERING_IRON_THERM
 Text GLabel 10325 6325 2    50   Input ~ 0
-SOLDERING_IRON_HEATER
+SOLDERING_IRON_HEATER_GND
 Wire Wire Line
 	10175 6575 10175 6325
@@
 	9900 11550 9900 11350
 Wire Wire Line
-	9900 11550 10375 11550
+	9900 11550 10250 11550
 $Comp
 L power:+24V #PWR0114
@@
 Text GLabel 7950 9950 0    50   Input ~ 0
 SOLDERING_IRON_THERM
-Wire Wire Line
-	10375 11950 10050 11950
-Wire Wire Line
-	10050 11950 10050 12050
 Wire Notes Line
 	450  1175 22800 1175
@@
 Text GLabel 1300 12000 0    50   Input ~ 0
 HOTAIR_THERM
-$Comp
-L Device:R R11
-U 1 1 5F8115BA
-P 3650 14075
-F 0 "R11" V 3650 14175 50  0000 R CNN
-F 1 "0R" V 3650 14075 50  0000 R CNN
-F 2 "Capacitors:0805" V 3580 14075 50  0001 C CNN
-F 3 "~" H 3650 14075 50  0001 C CNN
-	1    3650 14075
-	0    -1   -1   0
-$EndComp
 Wire Wire Line
 	3900 13375 3800 13375
@@
 	3800 13375 3800 13425
 Wire Wire Line
-	3900 14075 3800 14075
-$Comp
-L power:GND #PWR0129
-U 1 1 5F839D58
-P 2900 14225
-F 0 "#PWR0129" H 2900 13975 50  0001 C CNN
-F 1 "GND" H 2905 14052 50  0000 C CNN
-F 2 "" H 2900 14225 50  0001 C CNN
-F 3 "" H 2900 14225 50  0001 C CNN
-	1    2900 14225
-	1    0    0    -1
-$EndComp
-$Comp
-L Device:R R26
-U 1 1 5F8479CC
-P 9900 11850
-F 0 "R26" V 9800 11900 50  0000 R CNN
-F 1 "0R" V 9725 11900 50  0000 R CNN
-F 2 "Capacitors:0805" V 9830 11850 50  0001 C CNN
-F 3 "~" H 9900 11850 50  0001 C CNN
-	1    9900 11850
-	0    -1   -1   0
-$EndComp
-Wire Wire Line
-	10375 11850 10050 11850
-$Comp
-L power:GND #PWR0130
-U 1 1 5F864043
-P 9700 12150
-F 0 "#PWR0130" H 9700 11900 50  0001 C CNN
-F 1 "GND" H 9705 11977 50  0000 C CNN
-F 2 "" H 9700 12150 50  0001 C CNN
-F 3 "" H 9700 12150 50  0001 C CNN
-	1    9700 12150
-	1    0    0    -1
-$EndComp
-Wire Wire Line
-	9700 12150 9700 11850
-Wire Wire Line
-	9700 11850 9750 11850
+	10375 12050 10150 12050
 $Comp
 L Device:R R27
@@
 	1    0    0    -1
 $EndComp
-Wire Wire Line
-	3500 14075 2900 14075
-Wire Wire Line
-	2900 14075 2900 14225
 $Comp
 L Connector_Generic:Conn_01x04 J4
@@
 F 0 "D3" V 4254 8929 50  0000 L CNN
 F 1 "1N5819" V 4345 8929 50  0000 L CNN
-F 2 "Diode_THT:D_DO-41_SOD81_P10.16mm_Horizontal" H 4300 8675 50  0001 C CNN
+F 2 "Diode_SMD:D_MELF" H 4300 8675 50  0001 C CNN
 F 3 "http://www.vishay.com/docs/88525/1n5817.pdf" H 4300 8850 50  0001 C CNN
 	1    4300 8850
@@
 Wire Wire Line
 	16850 8850 16425 8850
-Wire Wire Line
-	10375 12050 10050 12050
-Connection ~ 10050 12050
-Wire Wire Line
-	10050 12050 10050 12150
 $Comp
 L Connector_Generic:Conn_01x06 J9
@@
 	0    -1   -1   0
 $EndComp
+Wire Wire Line
+	10150 11950 10375 11950
+Wire Wire Line
+	9900 11750 10250 11750
+Wire Wire Line
+	10375 11850 10250 11850
+Wire Wire Line
+	10250 11850 10250 11750
+Connection ~ 10250 11750
+Wire Wire Line
+	10250 11750 10375 11750
+Wire Wire Line
+	10375 11650 10250 11650
+Wire Wire Line
+	10250 11650 10250 11550
+Connection ~ 10250 11550
+Wire Wire Line
+	10250 11550 10375 11550
+Text GLabel 10150 12050 0    50   Input ~ 0
+THERM_GND
+Text GLabel 3725 14075 0    50   Input ~ 0
+THERM_GND
+Wire Wire Line
+	3725 14075 3900 14075
+Text GLabel 1725 13850 0    50   Input ~ 0
+THERM_GND
+$Comp
+L Device:R R9
+U 1 1 5FD30F23
+P 2000 13850
+F 0 "R9" V 2075 13900 50  0000 R CNN
+F 1 "0R" V 1900 13925 50  0000 R CNN
+F 2 "Capacitors:0805" V 1930 13850 50  0001 C CNN
+F 3 "~" H 2000 13850 50  0001 C CNN
+	1    2000 13850
+	0    -1   -1   0
+$EndComp
+$Comp
+L power:GND #PWR0112
+U 1 1 5FD31428
+P 2225 14025
+F 0 "#PWR0112" H 2225 13775 50  0001 C CNN
+F 1 "GND" H 2230 13852 50  0000 C CNN
+F 2 "" H 2225 14025 50  0001 C CNN
+F 3 "" H 2225 14025 50  0001 C CNN
+	1    2225 14025
+	1    0    0    -1
+$EndComp
+Wire Wire Line
+	1850 13850 1725 13850
+Wire Wire Line
+	2150 13850 2225 13850
+Wire Wire Line
+	2225 13850 2225 14025
 $EndSCHEMATC
