File: PCB/Hotair-soldering-station/main-pcb/hotair-soldering-station-main-pcb.sch (KiCad schematic (older format))
At the start: 89 parts, among them J1 230VAC_IN, J10 PA11, J11 PA12, J12 PA15, J13 ICP (goldpin r2,54), J2 main-board-conn, J3 EARTH_GND, J4 24V_IN (NS-25 r2,54), J5 PSUPPLY (PWZ-02S r.3,96), J6 HOTAIR_FAN (JST r,2,54)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

Commit message: PCB design update
Parts:
- C17, C18, C19: footprint Capacitors:0805 -> Capacitors:0603
- J10: value PA11 -> PB6
- J11: value PA12 -> PB4
- J12: value PA15 -> PB7
- R6: value 160R -> 320R
Connections:
- net +3V3: no longer U1.1
- net +5V: now also U1.1
- net BUZZER: now also U5.10 (PA4); no longer U5.18 (PA8)
- net FAN_PWM: now also U5.28 (PB5); no longer U5.20 (PA10)
- net HOTAIR_DOWN_SW: now also U5.15 (PB1); no longer U5.28 (PB5)
- net HOTAIR_FAN_DOWN_SW: now also U5.21 (PA11); no longer U5.2 (PF0)
- net HOTAIR_FAN_UP_SW: now also U5.20 (PA10); no longer U5.3 (PF1)
- net HOTAIR_HEATER_CTRL: now also U5.9 (PA3); no longer U5.10 (PA4)
- net HOTAIR_ON_SW: now also U5.22 (PA12); no longer U5.15 (PB1)
- net HOTAIR_REED_SW: now also U5.3 (PF1); no longer U5.30 (PB7)
- net HOTAIR_THERM: now also J7.1 (Pin_1)
- net HOTAIR_UP_SW: now also U5.18 (PA8); no longer U5.29 (PB6)
- net SOLDERING_IRON_THERM: no longer J7.1 (Pin_1)
- net SOLDER_DOWN_SW: now also U5.8 (PA2); no longer U5.26 (PB3)
- net SOLDER_ON_SW: now also U5.2 (PF0); no longer U5.14 (PB0)
- net SOLDER_UP_SW: now also U5.14 (PB0); no longer U5.27 (PB4)
- net SOLD_IRON_HEATER_CTRL: now also U5.26 (PB3); no longer U5.9 (PA3)
- net UART_DBG_TX: now also U5.19 (PA9); no longer U5.8 (PA2)
- net at R32.2, U6.2 (DQ): now also U5.25 (PA15); no longer U5.19 (PA9)
- net at J10.1 (Pin_1): now also U5.29 (PB6); no longer U5.21 (PA11)
- net at J11.1 (Pin_1): now also U5.27 (PB4); no longer U5.22 (PA12)
- net at J12.1 (Pin_1): now also U5.30 (PB7); no longer U5.25 (PA15)
Other:
- note added: "TIM14CH1 - Output compare (buzer)"
- note added: "TIM3_CH2 - PWM"
- moved on the sheet: J10, J11, J12
Changed lines of the file:
@@
-	1    0    0    -1
-$EndComp
-$Comp
-L power:+3V3 #PWR0101
-U 1 1 5F7DC810
-P 2350 6075
-F 0 "#PWR0101" H 2350 5925 50  0001 C CNN
-F 1 "+3V3" H 2365 6248 50  0000 C CNN
-F 2 "" H 2350 6075 50  0001 C CNN
-F 3 "" H 2350 6075 50  0001 C CNN
-	1    2350 6075
 	1    0    0    -1
 $EndComp
@@
 P 2350 6700
 F 0 "R6" H 2280 6654 50  0000 R CNN
-F 1 "160R" H 2280 6745 50  0000 R CNN
+F 1 "320R" H 2280 6745 50  0000 R CNN
 F 2 "Capacitors:0805" V 2280 6700 50  0001 C CNN
 F 3 "~" H 2350 6700 50  0001 C CNN
@@
 Wire Notes Line
 	12700 16075 12750 16075
-Text GLabel 16450 9550 0    50   Input ~ 0
+Text GLabel 18450 8950 2    50   Input ~ 0
 HOTAIR_UP_SW
-Text GLabel 16450 9450 0    50   Input ~ 0
+Text GLabel 16450 9150 0    50   Input ~ 0
 HOTAIR_DOWN_SW
-Text GLabel 16450 9350 0    50   Input ~ 0
-SOLDER_UP_SW
-Text GLabel 16450 9250 0    50   Input ~ 0
-SOLDER_DOWN_SW
-Text GLabel 16450 9150 0    50   Input ~ 0
-HOTAIR_ON_SW
-Text GLabel 16450 9050 0    50   Input ~ 0
-SOLDER_ON_SW
 Text GLabel 18450 8850 2    50   Input ~ 0
 7SEG_DIN
@@
 Text GLabel 18450 8750 2    50   Input ~ 0
 7SEG_LATCH
-Text GLabel 18450 8450 2    50   Input ~ 0
-SOLD_IRON_HEATER_CTRL
 Text GLabel 11925 9750 2    50   Input ~ 0
 THERM_IRON_ADC
 Text GLabel 18450 8150 2    50   Input ~ 0
 THERM_IRON_ADC
-Text GLabel 18450 8550 2    50   Input ~ 0
-HOTAIR_HEATER_CTRL
 $Comp
 L Device:R R7
@@
 	1    0    0    -1
 $EndComp
-Text GLabel 18450 8350 2    50   Input ~ 0
+Text GLabel 18450 9050 2    50   Input ~ 0
 UART_DBG_TX
 Wire Wire Line
@@
 	16850 9250 16450 9250
 Wire Wire Line
-	16450 9350 16850 9350
+	15450 9350 16850 9350
 Wire Wire Line
 	16450 9450 16850 9450
 Wire Wire Line
-	16850 9550 16450 9550
+	16850 9550 15450 9550
 Wire Wire Line
 	18450 8450 17950 8450
 Wire Wire Line
 	18450 8550 17950 8550
-Text GLabel 16450 9650 0    50   Input ~ 0
+Text GLabel 16425 8850 0    50   Input ~ 0
 HOTAIR_REED_SW
-Wire Wire Line
-	16450 9650 16850 9650
-Text GLabel 18450 8950 2    50   Input ~ 0
-BUZZER
 Wire Wire Line
 	18450 8950 17950 8950
@@
 Wire Wire Line
 	3900 14175 3750 14175
-Text GLabel 3750 13975 0    50   Input ~ 0
-SOLDERING_IRON_THERM
 Text Notes 775  13075 0    98   ~ 0
 HOTAIR connector\n
@@
 F 0 "C19" H 14665 6346 50  0000 L CNN
 F 1 "100n" H 14665 6255 50  0000 L CNN
-F 2 "Capacitors:0805" H 14588 6150 50  0001 C CNN
+F 2 "Capacitors:0603" H 14588 6150 50  0001 C CNN
 F 3 "~" H 14550 6300 50  0001 C CNN
 	1    14550 6300
@@
 F 0 "C18" H 14265 6346 50  0000 L CNN
 F 1 "100n" H 14265 6255 50  0000 L CNN
-F 2 "Capacitors:0805" H 14188 6150 50  0001 C CNN
+F 2 "Capacitors:0603" H 14188 6150 50  0001 C CNN
 F 3 "~" H 14150 6300 50  0001 C CNN
 	1    14150 6300
@@
 F 0 "C17" H 13815 6346 50  0000 L CNN
 F 1 "100n" H 13815 6255 50  0000 L CNN
-F 2 "Capacitors:0805" H 13738 6150 50  0001 C CNN
+F 2 "Capacitors:0603" H 13738 6150 50  0001 C CNN
 F 3 "~" H 13700 6300 50  0001 C CNN
 	1    13700 6300
@@
 Wire Wire Line
 	20550 9450 20550 9350
-Wire Wire Line
-	17950 9050 20150 9050
 $Comp
 L Device:R R32
@@
 Wire Wire Line
 	20150 9000 20150 9050
-Connection ~ 20150 9050
 Wire Wire Line
 	20150 9050 20250 9050
@@
 Wire Wire Line
 	20550 8650 20550 8750
-Text GLabel 18450 9150 2    50   Input ~ 0
-FAN_PWM
 Wire Wire Line
 	18450 9150 17950 9150
@@
 Text GLabel 1150 9900 0    50   Input ~ 0
 FAN_PWM
-Text GLabel 16425 8750 0    50   Input ~ 0
+Text GLabel 18450 9250 2    50   Input ~ 0
 HOTAIR_FAN_DOWN_SW
-Text GLabel 16425 8850 0    50   Input ~ 0
+Text GLabel 18450 9150 2    50   Input ~ 0
 HOTAIR_FAN_UP_SW
 Wire Wire Line
@@
 L Connector_Generic:Conn_01x01 J10
 U 1 1 5FC8B12E
-P 19150 9250
-F 0 "J10" H 19225 9250 50  0000 L CNN
-F 1 "PA11" H 19400 9250 50  0000 L CNN
-F 2 "My-Footprints:WIRE_PAD_1,3mm" H 19150 9250 50  0001 C CNN
-F 3 "~" H 19150 9250 50  0001 C CNN
-	1    19150 9250
-	1    0    0    -1
-$EndComp
-$Comp
-L Connector_Generic:Conn_01x01 J11
-U 1 1 5FC8CFCD
-P 19150 9350
-F 0 "J11" H 19225 9350 50  0000 L CNN
-F 1 "PA12" H 19400 9350 50  0000 L CNN
-F 2 "My-Footprints:WIRE_PAD_1,3mm" H 19150 9350 50  0001 C CNN
-F 3 "~" H 19150 9350 50  0001 C CNN
-	1    19150 9350
-	1    0    0    -1
+P 15250 9550
+F 0 "J10" H 15325 9550 50  0000 L CNN
+F 1 "PB6" H 15500 9550 50  0000 L CNN
+F 2 "My-Footprints:WIRE_PAD_1,3mm" H 15250 9550 50  0001 C CNN
+F 3 "~" H 15250 9550 50  0001 C CNN
+	1    15250 9550
+	-1   0    0    1
 $EndComp
 $Comp
 L Connector_Generic:Conn_01x01 J12
 U 1 1 5FC8D212
-P 19150 9650
-F 0 "J12" H 19225 9650 50  0000 L CNN
-F 1 "PA15" H 19400 9650 50  0000 L CNN
-F 2 "My-Footprints:WIRE_PAD_1,3mm" H 19150 9650 50  0001 C CNN
-F 3 "~" H 19150 9650 50  0001 C CNN
-	1    19150 9650
-	1    0    0    -1
-$EndComp
-Wire Wire Line
-	18950 9250 17950 9250
-Wire Wire Line
-	17950 9350 18950 9350
-Wire Wire Line
-	17950 9650 18950 9650
+P 15250 9650
+F 0 "J12" H 15325 9650 50  0000 L CNN
+F 1 "PB7" H 15500 9650 50  0000 L CNN
+F 2 "My-Footprints:WIRE_PAD_1,3mm" H 15250 9650 50  0001 C CNN
+F 3 "~" H 15250 9650 50  0001 C CNN
+	1    15250 9650
+	-1   0    0    1
+$EndComp
+Wire Wire Line
+	18450 9250 17950 9250
+Wire Wire Line
+	17950 9350 18450 9350
 $Comp
 L Connector_Generic:Conn_02x07_Counter_Clockwise J2
@@
 Wire Wire Line
 	2225 13850 2225 14025
+Text GLabel 18450 8550 2    50   Input ~ 0
+BUZZER
+Text GLabel 18450 8450 2    50   Input ~ 0
+HOTAIR_HEATER_CTRL
+Text GLabel 16450 9250 0    50   Input ~ 0
+SOLD_IRON_HEATER_CTRL
+Wire Wire Line
+	15450 9650 16850 9650
+Wire Wire Line
+	17950 9050 18450 9050
+Wire Wire Line
+	17950 9650 19875 9650
+Wire Wire Line
+	19875 9650 19875 9050
+Wire Wire Line
+	19875 9050 20150 9050
+Connection ~ 20150 9050
+Text GLabel 3750 13975 0    50   Input ~ 0
+HOTAIR_THERM
+$Comp
+L power:+5V #PWR0101
+U 1 1 5FE11A9C
+P 2350 6075
+F 0 "#PWR0101" H 2350 5925 50  0001 C CNN
+F 1 "+5V" H 2365 6248 50  0000 C CNN
+F 2 "" H 2350 6075 50  0001 C CNN
+F 3 "" H 2350 6075 50  0001 C CNN
+	1    2350 6075
+	1    0    0    -1
+$EndComp
+Text GLabel 18450 8350 2    50   Input ~ 0
+SOLDER_DOWN_SW
+Text GLabel 16425 8750 0    50   Input ~ 0
+SOLDER_ON_SW
+Text GLabel 16450 9050 0    50   Input ~ 0
+SOLDER_UP_SW
+Text GLabel 18450 9350 2    50   Input ~ 0
+HOTAIR_ON_SW
+Text GLabel 16450 9450 0    50   Input ~ 0
+FAN_PWM
+$Comp
+L Connector_Generic:Conn_01x01 J11
+U 1 1 5FC8CFCD
+P 15250 9350
+F 0 "J11" H 15325 9350 50  0000 L CNN
+F 1 "PB4" H 15500 9350 50  0000 L CNN
+F 2 "My-Footprints:WIRE_PAD_1,3mm" H 15250 9350 50  0001 C CNN
+F 3 "~" H 15250 9350 50  0001 C CNN
+	1    15250 9350
+	-1   0    0    1
+$EndComp
+Text Notes 15625 9975 0    50   ~ 0
+TIM3_CH2 - PWM
+Text Notes 15625 10075 0    50   ~ 0
+TIM14CH1 - Output compare (buzer)
 $EndSCHEMATC
