File: PCB/Hotair-soldering-station/main-pcb/hotair-soldering-station-main-pcb.kicad_pcb (KiCad board)
At the start: 2 copper layers, 90 parts, among them J1 230VAC_IN, J10 PA11, J11 PA12, J12 PA15, J13 ICP (goldpin r2,54), J2 main-board-conn, J3 EARTH_GND, J4 24V_IN (NS-25 r2,54), J5 PSUPPLY (PWZ-02S r.3,96), J6 HOTAIR_FAN (JST r,2,54), J7 HOTAIR_MEAS (JST r.2,5), J8 HOTAIR_HEATER (PWZ-02S r.3,96), J9 SOLD_IRON (r.2,54), Q1 BC817, Q2 BC817, Q3 BC817, Q4 BC807, Q5 IRLIZ44N, Q6 BT139-600, Q7 BC817, Q8 FP3055LP, Q9 BC817, U1 MOC3041M, U2 LMV324, U3 MP1584-Step-Down, U4 AMS1117-3.3, U5 STM32F030K6Tx, U6 DS18B20

Commit message: main pcb routing
Parts:
- removed R14, R9: 390R, Resistor_THT:R_Axial_DIN0414_L11.9mm_D4.5mm_P20.32mm_Horizontal
- added R33: 100R, Capacitors:0805, F.Cu at (87.5, 66.8)
- added R34: 100R, Capacitors:0805, F.Cu at (90.2, 66.0)
- R10, R15: value 390R -> 2x390R; footprint Resistor_THT:R_Axial_DIN0414_L11.9mm_D4.5mm_P20.32mm_Horizontal -> Resistor_THT:R_Axial_DIN0414_L11.9mm_D4.5mm_P15.24mm_Horizontal
- R12, R17: footprint Resistor_THT:R_Axial_DIN0414_L11.9mm_D4.5mm_P20.32mm_Horizontal -> Resistor_THT:R_Axial_DIN0414_L11.9mm_D4.5mm_P15.24mm_Horizontal
- U4: value AMS1117-3.3 -> AP1117-ADJ
- moved Q6 220.0 mm to (47.9, 69.3), turned to 90 degrees
- moved F3 206.7 mm to (60.1, 33.5), turned to 270 degrees
- moved R10 200.1 mm to (45.5, 79.6)
- moved J8 197.7 mm to (71.8, 54.0), turned to 90 degrees
- moved U1 194.2 mm to (58.3, 93.3), turned to 90 degrees
- moved R6 192.2 mm to (54.9, 96.0), turned to 180 degrees
- moved C7 191.7 mm to (74.7, 66.9), turned to 180 degrees
- moved R12 189.2 mm to (54.2, 59.6), turned to 270 degrees
- moved R3 187.4 mm to (54.9, 97.9)
- moved Q1 185.2 mm to (58.4, 96.6), turned to 90 degrees
- moved R17 183.0 mm to (59.4, 61.0)
- moved C5 177.7 mm to (74.2, 79.6), turned to 180 degrees
- moved R15 172.6 mm to (74.9, 73.0), turned to 180 degrees
- moved J6 144.7 mm to (40.6, 101.5), turned to 90 degrees
- moved J3 135.1 mm to (79.4, 30.9), turned to 180 degrees
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Connections:
- C14 pad 2: GND -> Net-(C14-Pad2)
- C15 pad 2: GND -> Net-(C14-Pad2)
- Q8 pad 3: Net-(Q8-Pad3) -> Net-(C14-Pad2)
- R27 pad 1: Net-(Q8-Pad3) -> Net-(C14-Pad2)
- U4 pad 1: GND -> Net-(R33-Pad1)
- U5 pad 31: (no net) -> GND
Routing:
- net AC_230(N): track 0.00 -> 87.8 mm
- net Net-(Q6-Pad3): track 0.00 -> 47.6 mm
- net Net-(J8-Pad1): track 0.00 -> 44.7 mm
- net Net-(C14-Pad2): track 0.00 -> 43.0 mm
- net GND: track 0.00 -> 32.1 mm, vias 0 -> 1
- net Net-(F1-Pad1): track 0.00 -> 31.7 mm
- net +24V: track 0.00 -> 24.3 mm
- net +3V3: track 0.00 -> 19.6 mm
- net AC_230(L): track 0.00 -> 18.9 mm
- net Net-(R10-Pad1): track 0.00 -> 17.1 mm
- net Net-(F3-Pad2): track 0.00 -> 14.7 mm
- net Net-(F2-Pad2): track 0.00 -> 12.1 mm
- net Net-(J1-Pad1): track 0.00 -> 10.8 mm
- net Net-(C5-Pad1): track 0.00 -> 6.92 mm
- net Net-(C7-Pad1): track 0.00 -> 5.97 mm
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- added copper zone on F.Cu, net GND
Other:
- board outline added: 95.1 x 100.5 mm
- net class 230V added: clearance 3, trace_width 0.25, via_dia 0.8, via_drill 0.4
- net class Default: clearance 0.2 -> 0.5
- rule trace_clearance: 0.2 -> 0.5

Commit message: PCB desingn update
Parts:
- removed R11, R26: 0R, Capacitors:0805
- added R9: 0R, Capacitors:0805, F.Cu at (60.8, 109.6)
- C10, C11, C14, C15, C16, C3, C5, C7, C8, C9, D5, F1, F2, F3, J2, J6, J7, J9, L1, LS1, Q5, Q8, R10, R12, R15, R17, U1, U3, U6: moved to B.Cu
- D3: footprint Diode_THT:D_DO-41_SOD81_P10.16mm_Horizontal -> Diode_SMD:D_MELF
- Q6: footprint Package_TO_SOT_THT:TO-220-3_Vertical -> My-Footprints:TO-220-3_Vertical; moved to B.Cu
- moved R2 110.8 mm to (48.1, 104.6), turned to 0 degrees
- moved R5 109.2 mm to (48.3, 109.6), turned to 0 degrees
- moved C1 107.1 mm to (48.9, 106.2), turned to 180 degrees
- moved C16 94.5 mm to (49.9, 103.3), turned to 90 degrees
- moved C4 92.2 mm to (67.4, 100.1)
- moved D4 92.2 mm to (70.8, 108.6)
- moved R13 92.2 mm to (67.5, 97.1)
- moved R16 92.2 mm to (70.8, 97.4)
- moved R18 92.2 mm to (71.9, 105.6)
- moved R7 92.2 mm to (67.5, 102.4)
- moved C12 91.4 mm to (45.5, 102.9), turned to 90 degrees
- moved U2 90.5 mm to (54.6, 104.1)
- moved R21 90.2 mm to (45.7, 100.3)
- moved R19 90.0 mm to (47.2, 102.9), turned to 270 degrees
- moved R23 88.5 mm to (49.0, 100.3)
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Connections:
- J7 pad 2: Net-(J7-Pad2) -> THERM_GND
- J9 pad 2: SOLDERING_IRON_HEATER -> +24V
- J9 pad 3: SOLDERING_IRON_THERM -> SOLDERING_IRON_HEATER_GND
- J9 pad 4: Net-(J9-Pad4) -> SOLDERING_IRON_HEATER_GND
- J9 pad 5: GND -> SOLDERING_IRON_THERM
- J9 pad 6: GND -> THERM_GND
- Q8 pad 2: SOLDERING_IRON_HEATER -> SOLDERING_IRON_HEATER_GND
- U2 pad 10: Net-(C1-Pad1) -> Net-(C4-Pad1)
- U2 pad 5: Net-(C4-Pad1) -> Net-(C1-Pad1)
- U2 pad 6: Net-(R13-Pad2) -> Net-(C4-Pad2)
- U2 pad 7: Net-(R16-Pad2) -> Net-(C4-Pad1)
- U2 pad 8: Net-(C4-Pad1) -> Net-(R16-Pad2)
- U2 pad 9: Net-(C4-Pad2) -> Net-(R13-Pad2)
Routing:
- net +24V: track 24.3 -> 135.8 mm
- net Net-(C14-Pad2): track 43.0 -> 107.1 mm
- net AC_230(N): track 87.8 -> 129.0 mm
- net FAN_SUPPLY: track 0.00 -> 30.7 mm
- net GND: track 32.1 -> 2.16 mm, vias 1 -> 2
- net +5V: track 4.85 -> 33.1 mm
- net Net-(D1-Pad1): track 0.00 -> 20.7 mm
- net AC_230(L): track 18.9 -> 39.2 mm
- net Net-(C5-Pad1): track 6.92 -> 25.9 mm
- net Net-(C6-Pad2): track 0.00 -> 17.7 mm
- net Net-(C6-Pad1): track 0.00 -> 12.1 mm
- net Net-(Q3-Pad2): track 0.00 -> 10.5 mm, vias 0 -> 1
- net SOLDERING_IRON_HEATER_GND: track 0.00 -> 10.2 mm
- net Net-(F2-Pad2): track 12.1 -> 21.9 mm
- net Net-(J8-Pad1): track 44.7 -> 53.3 mm
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- added copper zone on B.Cu, net GND
Other:
- board size 95.1 x 100.5 mm -> 89.4 x 90.9 mm
- net class 230V: trace_width 0.25 -> 0.2

Commit message: PCB design update
Parts:
- C16: moved to F.Cu
- C17, C19: footprint Capacitors:0805 -> Capacitors:0603
- C18: footprint Capacitors:0805 -> Capacitors:0603; moved to B.Cu
- R6: value 160R -> 320R
- moved LS1 97.2 mm to (41.1, 101.5), turned to 0 degrees
- moved Q9 93.2 mm to (51.7, 106.4), turned to 180 degrees
- moved R31 92.2 mm to (55.8, 107.3)
- moved D6 48.5 mm to (82.2, 97.8), turned to 270 degrees
- moved R9 23.9 mm to (83.4, 101.9), turned to 180 degrees
- moved R21 21.9 mm to (66.5, 93.6), turned to 270 degrees
- moved R30 19.1 mm to (78.9, 96.1), turned to 0 degrees
- moved C13 18.5 mm to (67.3, 96.0)
- moved R23 18.5 mm to (67.3, 97.8)
- moved R29 18.4 mm to (78.1, 98.7)
- moved R28 18.4 mm to (79.9, 98.7)
- moved U2 18.4 mm to (72.9, 101.9)
- moved R19 17.8 mm to (64.8, 99.6)
- moved C12 17.7 mm to (62.9, 99.6)
- moved R5 17.0 mm to (64.6, 105.2), turned to 90 degrees
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Connections:
- J7 pad 1: SOLDERING_IRON_THERM -> HOTAIR_THERM
- R2 pad 1: (no net) -> HOTAIR_THERM
- U1 pad 1: +3V3 -> +5V
- U5 pad 10: HOTAIR_HEATER_CTRL -> BUZZER
- U5 pad 14: SOLDER_ON_SW -> SOLDER_UP_SW
- U5 pad 15: HOTAIR_ON_SW -> HOTAIR_DOWN_SW
- U5 pad 18: BUZZER -> HOTAIR_UP_SW
- U5 pad 19: Net-(R32-Pad2) -> UART_DBG_TX
- U5 pad 2: HOTAIR_FAN_DOWN_SW -> SOLDER_ON_SW
- U5 pad 20: FAN_PWM -> HOTAIR_FAN_UP_SW
- U5 pad 21: Net-(J10-Pad1) -> HOTAIR_FAN_DOWN_SW
- U5 pad 22: Net-(J11-Pad1) -> HOTAIR_ON_SW
- U5 pad 25: Net-(J12-Pad1) -> Net-(R32-Pad2)
- U5 pad 26: SOLDER_DOWN_SW -> SOLD_IRON_HEATER_CTRL
- U5 pad 27: SOLDER_UP_SW -> Net-(J11-Pad1)
- U5 pad 28: HOTAIR_DOWN_SW -> FAN_PWM
- U5 pad 29: HOTAIR_UP_SW -> Net-(J10-Pad1)
- U5 pad 3: HOTAIR_FAN_UP_SW -> HOTAIR_REED_SW
- U5 pad 30: HOTAIR_REED_SW -> Net-(J12-Pad1)
- U5 pad 8: UART_DBG_TX -> SOLDER_DOWN_SW
- U5 pad 9: SOLD_IRON_HEATER_CTRL -> HOTAIR_HEATER_CTRL
Routing:
- net +3V3: track 19.6 -> 144.8 mm, vias 0 -> 3
- net +5V: track 33.1 -> 142.0 mm, vias 0 -> 2
- net SOLDERING_IRON_THERM: track 0.00 -> 79.8 mm, vias 0 -> 3
- net THERM_GND: track 0.00 -> 64.8 mm, vias 0 -> 1
- net HOTAIR_HEATER_CTRL: track 0.00 -> 62.9 mm
- net BUZZER: track 0.00 -> 61.1 mm
- net HOTAIR_THERM: track 0.00 -> 54.7 mm, vias 0 -> 1
- net SOLDER_ON_SW: track 0.00 -> 39.0 mm, vias 0 -> 1
- net RST: track 0.00 -> 36.3 mm, vias 0 -> 1
- net HOTAIR_ON_SW: track 0.00 -> 35.0 mm
- net THERM_HOTAIR_ADC: track 0.00 -> 33.4 mm
- net 7SEG_CLK: track 0.00 -> 30.9 mm
- net HOTAIR_FAN_DOWN_SW: track 0.00 -> 28.3 mm
- net FAN_PWM: track 0.00 -> 27.1 mm, vias 0 -> 2
- net THERM_IRON_ADC: track 0.00 -> 26.8 mm
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Other:
- net class Default: clearance 0.5 -> 0.7
- rule trace_clearance: 0.5 -> 0.7
