File: PCB/front-pcb/Hotair-soldering-station.kicad_pcb (KiCad board)
At the start: 2 copper layers, 70 x 120 mm, 60 parts, among them J2 main-board-conn, J3 hot_on, J4 solder_on, Q1 BC817, Q10 BC807, Q11 BC807, Q12 BC807, Q13 BC807, Q14 BC807, Q2 BC817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

Commit message: LED display, buzzer and PWM done in SW. Some HW bugs fixed.
Connections:
- U1 pad 10: GND -> +3V3
- U2 pad 10: GND -> +3V3
Routing:
- net +3V3: track 322.1 -> 357.2 mm, vias 8 -> 10
Changed lines of the file:
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@@
     (thickness 1.6)
     (drawings 18)
-    (tracks 411)
+    (tracks 425)
     (zones 0)
     (modules 60)
@@
   )
   (setup
-    (last_trace_width 0.25)
+    (last_trace_width 0.6)
     (user_trace_width 0.4)
     (user_trace_width 0.5)
@@
     (add_net "Net-(R9-Pad2)")
     (add_net "Net-(U1-Pad9)")
+    (add_net "Net-(U2-Pad6)")
+    (add_net "Net-(U2-Pad7)")
+    (add_net "Net-(U2-Pad9)")
     (add_net SEG_A)
     (add_net SEG_B)
@@
       (net 9 7SEG_CLK) (solder_mask_margin 0.1016))
     (pad 10 smd rect (at 3.175 2.79908) (size 0.59944 1.19888) (layers B.Cu B.Paste B.Mask)
-      (net 7 GND) (solder_mask_margin 0.1016))
+      (net 11 +3V3) (solder_mask_margin 0.1016))
     (pad 9 smd rect (at 4.445 2.79908) (size 0.59944 1.19888) (layers B.Cu B.Paste B.Mask)
       (solder_mask_margin 0.1016))
@@
       (net 9 7SEG_CLK) (solder_mask_margin 0.1016))
     (pad 10 smd rect (at 3.175 2.79908) (size 0.59944 1.19888) (layers B.Cu B.Paste B.Mask)
-      (net 7 GND) (solder_mask_margin 0.1016))
+      (net 11 +3V3) (solder_mask_margin 0.1016))
     (pad 9 smd rect (at 4.445 2.79908) (size 0.59944 1.19888) (layers B.Cu B.Paste B.Mask)
       (net 48 "Net-(U1-Pad9)") (solder_mask_margin 0.1016))
@@
   (segment (start 60.47058 127.35226) (end 60.59932 127.22352) (width 0.7) (layer B.Cu) (net 11))
   (segment (start 60.47058 128.43256) (end 60.47058 127.35226) (width 0.7) (layer B.Cu) (net 11))
-  (segment (start 64.11468 130.78968) (end 60.59932 127.22352) (width 0.7) (layer B.Cu) (net 11))
   (segment (start 60.59932 127.22352) (end 59.4614 126.1364) (width 0.7) (layer B.Cu) (net 11))
   (segment (start 59.32424 39.46144) (end 59.13628 39.27348) (width 0.8) (layer F.Cu) (net 11))
@@
   (segment (start 59.66968 39.80688) (end 59.13628 39.27348) (width 0.8) (layer F.Cu) (net 11))
   (segment (start 63.7794 39.80688) (end 59.66968 39.80688) (width 0.8) (layer F.Cu) (net 11))
+  (via (at 76.962 132.588) (size 0.8) (drill 0.4) (layers F.Cu B.Cu) (net 11))
+  (segment (start 76.0984 130.78968) (end 76.0984 131.7244) (width 0.6) (layer B.Cu) (net 11))
+  (segment (start 76.0984 131.7244) (end 76.962 132.588) (width 0.6) (layer B.Cu) (net 11))
+  (via (at 64.11468 130.78968) (size 0.8) (drill 0.4) (layers F.Cu B.Cu) (net 11))
+  (segment (start 76.962 132.588) (end 65.913 132.588) (width 0.6) (layer F.Cu) (net 11))
+  (segment (start 65.913 132.588) (end 64.11468 130.78968) (width 0.6) (layer F.Cu) (net 11))
+  (segment (start 45.8724 133.07568) (end 45.8724 133.8834) (width 0.6) (layer B.Cu) (net 11))
+  (segment (start 45.8724 133.8834) (end 45.847 133.858) (width 0.6) (layer B.Cu) (net 11))
+  (segment (start 45.847 133.858) (end 45.847 131.318) (width 0.6) (layer B.Cu) (net 11))
+  (segment (start 45.847 131.318) (end 46.228 130.937) (width 0.6) (layer B.Cu) (net 11))
+  (segment (start 63.96736 130.937) (end 64.11468 130.78968) (width 0.6) (layer B.Cu) (net 11))
+  (segment (start 60.47058 130.91842) (end 60.452 130.937) (width 0.6) (layer B.Cu) (net 11))
+  (segment (start 60.47058 128.43256) (end 60.47058 130.91842) (width 0.6) (layer B.Cu) (net 11))
+  (segment (start 46.228 130.937) (end 60.452 130.937) (width 0.6) (layer B.Cu) (net 11))
+  (segment (start 60.452 130.937) (end 63.96736 130.937) (width 0.6) (layer B.Cu) (net 11))
   (segment (start 51.8414 115.17376) (end 51.8414 116.8306) (width 0.7) (layer B.Cu) (net 12))
   (segment (start 52.7914 120.17244) (end 52.7304 120.23344) (width 0.8) (layer B.Cu) (net 13))
