File: PCB/V1.1/main-pcb/hotair-soldering-station-main-pcb (1).kicad_sch (KiCad schematic)
At the start: 96 parts, among them J1 230VAC_IN, J10 SOLD_IRON (r.2,54), J11 LCD_CON2 (JST r.2.0), J12 LCD_CON1 (JST r.2.0), J13 ICP (goldpin r2,54), J2 FRONT_PANEL (IDC r. 2,54), J3 EARTH_GND, J4 24V_IN (NS-25 r2,54), J5 PSUPPLY (PWZ-02S r.3,96), J6 HOTAIR_FAN (JST r,2,54), J7 HOTAIR_MEAS (JST r.2,5), J8 HOTAIR_HEATER (PWZ-02S r.3,96), J9 SOLD_IRON (r.2,54), Q1 BC817, Q10 FP3055LP, Q11 BC817, Q2 BC807, Q3 BC817, Q4 Q_PMOS_GDS, Q5 BC817, Q6 BT139-600, Q7 BC817, Q8 FP3055LP, Q9 BC817, U1 MOC3041M, U2 MAX31855KASA, U3 MP1584-Step-Down, U4 AP1117-ADJ, U6 LM358, U7 MAX31855KASA, U8 STM32F103C6Tx

Commit message: Routing PCB, front panel design progress
Parts:
- removed C17: 100n, Capacitors:0603, symbol Device:C
- C9: footprint Capacitors:0603 -> Capacitor_SMD:C_0603_1608Metric
- R27: footprint Capacitors:0805 -> Resistor_THT:R_Axial_DIN0204_L3.6mm_D1.6mm_P1.90mm_Vertical
Connections:
- net MAX31855_IRON_WEP_CS is gone; now on net MAX31855_IRON_CS: U7.6 (~{CS})
- net AC_230(N): no longer J5.2 (Pin_2)
- net GND: now also J2.14 (Pin_14), U8.44 (BOOT0); no longer J2.2 (Pin_2)
- net HOTAIR_DOWN_SW: now also J2.2 (Pin_2), U8.10 (PA0); no longer J2.11 (Pin_11), U8.27 (PB14)
- net HOTAIR_FAN_ADC: now also U8.11 (PA1); no longer U8.10 (PA0)
- net HOTAIR_FAN_DOWN_SW: now also J2.11 (Pin_11); no longer J2.9 (Pin_9)
- net HOTAIR_FAN_UP_SW: now also J2.13 (Pin_13); no longer J2.8 (Pin_8)
- net HOTAIR_ON_SW: now also J2.12 (Pin_12); no longer J2.13 (Pin_13)
- net HOTAIR_TEMP_ADC: now also U8.19 (PB1); no longer U8.11 (PA1)
- net IRON_T12_MOTION_SW: now also U8.27 (PB14); no longer U8.19 (PB1)
- net LCD_D5: now also J12.2 (Pin_2); no longer J12.4 (Pin_4)
- net LCD_D6: now also J12.1 (Pin_1); no longer J12.5 (Pin_5)
- net LCD_D7: now also J11.5 (Pin_5); no longer J12.6 (Pin_6)
- net LCD_EN: now also J12.4 (Pin_4); no longer J12.2 (Pin_2)
- net LCD_RS: now also J12.6 (Pin_6); no longer J11.5 (Pin_5)
- net LCD_RW: now also J12.5 (Pin_5); no longer J12.1 (Pin_1)
- net MAX31855_HOTAIR_CS: now also U8.14 (PA4); no longer U8.13 (PA3)
- net MAX31855_IRON_CS: now also U8.13 (PA3); no longer U8.14 (PA4)
- net MENU_UP_SW: now also J2.8 (Pin_8); no longer J2.3 (Pin_3)
- net SOLDER_ON_SW: now also J2.9 (Pin_9); no longer J2.14 (Pin_14)
- net SOLDER_SELECT_SW: now also J2.3 (Pin_3); no longer J2.12 (Pin_12)
Other:
- note added: "VDD pins: 1x 100nF + 1x10 µF Vbat pin: 100n VDDa pin: 1x100n + 1x1µF"
- moved on the sheet: J12
